Commit message: update model URDF with collision

File: description/models/diff_drive/model.urdf (robot description, URDF)
Before this commit: robot sam_bot, 3 links, 2 joints
Links:
- link base_link: geometry collision box size=${base_length} ${base_width} ${base_height}; visual box size=${base_length} ${base_width} ${base_height}
- link front_caster: geometry collision sphere radius=${(wheel_radius+wheel_zoff-(base_height/2))}; visual sphere radius=${(wheel_radius+wheel_zoff-(base_height/2))}

Commit message: #22 update with real values

File: description/models/diff_drive/model.urdf (robot description, URDF)
Before this commit: robot sam_bot, 3 links, 2 joints
Joints:
- joint caster_joint: origin xyz=${caster_xoff} 0.0 ${-(base_height/2)} rpy=0 0 0 -> xyz=${-caster_xoff} 0.0 ${-(base_height/2)} rpy=0 0 0
