Commit message: #22, #23

File: description/models/diff_drive/model.xacro (robot description, xacro)
@@ -1,4 +1,4 @@
 <?xml version="1.0"?>
-<robot name="sam_bot" xmlns:xacro="http://ros.org/wiki/xacro">
+<robot name="lego_bot" xmlns:xacro="http://ros.org/wiki/xacro">
     <!-- Define robot constants -->
     <!-- stud=0.008, w=13, l=17, h=14 -->
@@ -34,4 +34,11 @@
         </inertial>
     </xacro:macro>
+    <!-- dummy link without inertia for usage with KDL -->
+    <!-- <link name="base_link_without_inertia"/>
+    <joint name="base_link_without_inertia_joint" type="fixed">
+        <parent link="base_link_without_inertia"/>
+        <child link="base_link"/>
+        <origin xyz="0.0 0.0 0.0" rpy="0 0 0"/>
+    </joint> -->
     <!-- Robot Base -->
     <link name="base_link">
