Commit message: add gazebo world and new models

File: description/models/diff_drive/gazebo.xacro (robot description, xacro)
@@ -26,3 +26,9 @@
   </plugin>
 </gazebo>
+<!-- TODO do we need this????? -->
+<!-- <gazebo>
+  <plugin name="joint_state_publisher" filename="libgazebo_ros_joint_state_publisher.so">
+    <joint_name>drivewhl_l_joint, drivewhl_r_joint</joint_name>
+  </plugin>
+</gazebo> -->
 </robot>

File: description/models/diff_drive/model.xacro (robot description, xacro)
@@ -35,12 +35,12 @@
     </xacro:macro>
     <!-- dummy link without inertia for usage with KDL -->
-    <!-- <link name="base_link_without_inertia"/>
-    <joint name="base_link_without_inertia_joint" type="fixed">
-        <parent link="base_link_without_inertia"/>
-        <child link="base_link"/>
+    <!-- <link name="base_center_link_without_inertia"/>
+    <joint name="base_center_link_without_inertia_joint" type="fixed">
+        <parent link="base_center_link_without_inertia"/>
+        <child link="base_center_link"/>
         <origin xyz="0.0 0.0 0.0" rpy="0 0 0"/>
     </joint> -->
     <!-- Robot Base -->
-    <link name="base_link">
+    <link name="base_center_link">
         <visual>
             <geometry>
@@ -56,12 +56,12 @@
             </geometry>
         </collision>
-        <xacro:box_inertia m="15" w="${base_width}" d="${base_length}" h="${base_height}"/>
+        <xacro:box_inertia m="1" w="${base_width}" d="${base_length}" h="${base_height}"/>
     </link>
     <!-- Robot Footprint -->
-    <link name="base_footprint"/>
+    <link name="base_link"/>
     <joint name="base_joint" type="fixed">
         <parent link="base_link"/>
-        <child link="base_footprint"/>
-        <origin xyz="0.0 0.0 ${-(wheel_radius+wheel_zoff)}" rpy="0 0 0"/>
+        <child link="base_center_link"/>
+        <origin xyz="0.0 0.0 ${wheel_radius+wheel_zoff}" rpy="0 0 0"/>
     </joint>
     <!-- Wheels -->
@@ -83,8 +83,8 @@
             </geometry>
         </collision>
-        <xacro:cylinder_inertia m="0.5" r="${wheel_radius}" h="${wheel_width}"/>
+        <xacro:cylinder_inertia m="0.25" r="${wheel_radius}" h="${wheel_width}"/>
         </link>
         <joint name="${prefix}_joint" type="continuous">
-            <parent link="base_link"/>
+            <parent link="base_center_link"/>
             <child link="${prefix}_link"/>
             <origin xyz="${x_reflect*wheel_xoff} ${y_reflect*(base_width/2+wheel_ygap)} ${-wheel_zoff}" rpy="0 0 0"/>
@@ -110,8 +110,8 @@
             </geometry>
         </collision>
-        <xacro:sphere_inertia m="0.5" r="${(wheel_radius+wheel_zoff-(base_height/2))}"/>
+        <xacro:sphere_inertia m="0.25" r="${(wheel_radius+wheel_zoff-(base_height/2))}"/>
     </link>
     <joint name="caster_joint" type="fixed">
-        <parent link="base_link"/>
+        <parent link="base_center_link"/>
         <child link="front_caster"/>
         <origin xyz="${-caster_xoff} 0.0 ${-(base_height/2)}" rpy="0 0 0"/>
